File: esperimental.sch (KiCad schematic (older format))
At the start: 10 parts, among them P1 CONN_01X01, P2 CONN_01X01

Commit message: first draft of probably millable board
* adapt schematic slightly for easier production
* fix ESP8266 footprint to no longer include unnecessary drill holes
* add a ground fill
Parts:
- YOL0: footprint ESP8266:ESP-07v2 -> ESP8266SMD:ESP-07v2_smd
Connections:
- wire segments 24 -> 20
- no-connect marks 7 -> 6
Other:
- moved on the sheet: PINHDR0
Changed lines of the file:
@@
 LIBS:contrib
 LIBS:valves
-LIBS:ESP8266
+LIBS:esperimental-cache
 EELAYER 25 0
 EELAYER END
@@
 F 0 "YOL0" H 6000 4578 50  0000 C CNN
 F 1 "ESP-07v2" H 6000 4487 50  0000 C CNN
-F 2 "ESP8266:ESP-07v2" H 6000 3500 50  0001 C CNN
+F 2 "ESP8266SMD:ESP-07v2_smd" H 6000 3500 50  0001 C CNN
 F 3 "" H 6000 3500 50  0001 C CNN
 	1    6000 3500
@@
 L CONN_01X03 PINHDR0
 U 1 1 576EF38A
-P 7800 3050
-F 0 "PINHDR0" H 7878 3091 50  0000 L CNN
-F 1 "CONN_01X03" H 7878 3000 50  0000 L CNN
-F 2 "Pin_Headers:Pin_Header_Straight_1x03" H 7800 3050 50  0001 C CNN
-F 3 "" H 7800 3050 50  0000 C CNN
-	1    7800 3050
-	1    0    0    -1
-$EndComp
-$Comp
-L GND #PWR01
-U 1 1 576EF40C
-P 7400 2950
-F 0 "#PWR01" H 7400 2700 50  0001 C CNN
-F 1 "GND" H 7405 2777 50  0000 C CNN
-F 2 "" H 7400 2950 50  0000 C CNN
-F 3 "" H 7400 2950 50  0000 C CNN
-	1    7400 2950
-	1    0    0    -1
+P 8350 3300
+F 0 "PINHDR0" H 8428 3341 50  0000 L CNN
+F 1 "CONN_01X03" H 8428 3250 50  0000 L CNN
+F 2 "Pin_Headers:Pin_Header_Straight_1x03" H 8350 3300 50  0001 C CNN
+F 3 "" H 8350 3300 50  0000 C CNN
+	1    8350 3300
+	1    0    0    1
 $EndComp
 NoConn ~ 5100 3300
@@
 NoConn ~ 5100 3600
 NoConn ~ 5100 3700
-NoConn ~ 5100 3800
 NoConn ~ 6900 3400
 NoConn ~ 6900 3500
@@
 	7300 3350 7250 3350
 Wire Wire Line
-	6900 3300 7600 3300
-Wire Wire Line
-	7600 3300 7600 3150
-Wire Wire Line
-	7600 3050 7500 3050
-Wire Wire Line
-	7500 3050 7500 3200
-Wire Wire Line
-	7500 3200 6900 3200
-Wire Wire Line
-	7600 2950 7400 2950
-Wire Wire Line
 	7250 3700 7200 3700
 Wire Wire Line
@@
 $EndComp
 Wire Wire Line
-	3950 3550 3950 2600
+	3950 2600 3950 3550
 Wire Wire Line
 	3950 2600 7250 2600
@@
 	1    0    0    -1
 $EndComp
+$Comp
+L PWR_FLAG #FLG04
+U 1 1 576FC0D0
+P 3750 3950
+F 0 "#FLG04" H 3750 4045 50  0001 C CNN
+F 1 "PWR_FLAG" H 3750 4130 50  0000 C CNN
+F 2 "" H 3750 3950 50  0000 C CNN
+F 3 "" H 3750 3950 50  0000 C CNN
+	1    3750 3950
+	1    0    0    -1
+$EndComp
+$Comp
+L PWR_FLAG #FLG05
+U 1 1 576FC0F8
+P 3700 3050
+F 0 "#FLG05" H 3700 3145 50  0001 C CNN
+F 1 "PWR_FLAG" H 3700 3230 50  0000 C CNN
+F 2 "" H 3700 3050 50  0000 C CNN
+F 3 "" H 3700 3050 50  0000 C CNN
+	1    3700 3050
+	-1   0    0    1
+$EndComp
+Wire Wire Line
+	6900 3200 8150 3200
+Wire Wire Line
+	6900 3300 8150 3300
+$Comp
+L GND #PWR?
+U 1 1 576FC696
+P 8150 3400
+F 0 "#PWR?" H 8150 3150 50  0001 C CNN
+F 1 "GND" H 8150 3250 50  0000 C CNN
+F 2 "" H 8150 3400 50  0000 C CNN
+F 3 "" H 8150 3400 50  0000 C CNN
+	1    8150 3400
+	1    0    0    -1
+$EndComp
